Commit message: Our own changes to the xacro files

File: robots/youbot_base_only.urdf.xacro (robot description, xacro)
@@ -25,7 +25,3 @@
        is the world frame). For more, see http://www.ros.org/wiki/xacro -->
   <xacro:youbot_base name="base"/>
-  <!-- base laser front -->
-  <xacro:hokuyo_urg04_laser name="base_laser_front" parent="base" ros_topic="scan_front" update_rate="10" min_angle="-1.57" max_angle="1.57">
-    <origin xyz="0.3 0 -0.03" rpy="0 0 0"/>
-  </xacro:hokuyo_urg04_laser>
 </robot>

File: urdf/common.xacro (robot description, xacro)
@@ -1,4 +1,4 @@
 <?xml version="1.0"?>
-<robot>
+<robot xmlns:xacro="http://ros.org/wiki/xacro">
 	<property name="M_PI" value="3.1415926535897931" />
 	<!-- Casters -->

File: urdf/youbot_arm/limits.urdf.xacro (robot description, xacro)
@@ -2,30 +2,30 @@
 <robot xmlns:xacro="http://ros.org/wiki/xacro">>
 	<!-- common properties -->
-	<property name="M_PI" value="3.1415926535897931" />
-	<property name="threshold" value="0.01" />
+	<xacro:property name="M_PI" value="3.1415926535897931" />
+	<xacro:property name="threshold" value="0.01" />
 	<!-- arm limits positions (deg) -->
-	<property name="joint_1_limit" value="${M_PI * (169 + 169) / 180}" />
-	<property name="joint_2_limit" value="${M_PI * (90 + 65) / 180}" />
-	<property name="joint_3_limit" value="${M_PI * (146 + 151) / 180}" />
-	<property name="joint_4_limit" value="${M_PI * (102.5 + 102.5) / 180}" />
-	<property name="joint_5_limit" value="${M_PI * (167.5 + 167.5) / 180}" />
-	<property name="joint_1_limit_soft" value="${joint_1_limit - threshold}" />
-	<property name="joint_2_limit_soft" value="${joint_2_limit - threshold}" />
-	<property name="joint_3_limit_soft" value="${joint_3_limit - threshold}" />
-	<property name="joint_4_limit_soft" value="${joint_4_limit - threshold}" />
-	<property name="joint_5_limit_soft" value="${joint_5_limit - threshold}" />
+	<xacro:property name="joint_1_limit" value="${M_PI * (169 + 169) / 180}" />
+	<xacro:property name="joint_2_limit" value="${M_PI * (90 + 65) / 180}" />
+	<xacro:property name="joint_3_limit" value="${M_PI * (146 + 151) / 180}" />
+	<xacro:property name="joint_4_limit" value="${M_PI * (102.5 + 102.5) / 180}" />
+	<xacro:property name="joint_5_limit" value="${M_PI * (167.5 + 167.5) / 180}" />
+	<xacro:property name="joint_1_limit_soft" value="${joint_1_limit - threshold}" />
+	<xacro:property name="joint_2_limit_soft" value="${joint_2_limit - threshold}" />
+	<xacro:property name="joint_3_limit_soft" value="${joint_3_limit - threshold}" />
+	<xacro:property name="joint_4_limit_soft" value="${joint_4_limit - threshold}" />
+	<xacro:property name="joint_5_limit_soft" value="${joint_5_limit - threshold}" />
 	<!-- dynamic properties : mass (kg) Alu data sheet -->
-	<property name="link_0_mass" value="0.961" />
-	<property name="link_1_mass" value="1.390" />
-	<property name="link_2_mass" value="1.318" />
-	<property name="link_3_mass" value="0.821" />
-	<property name="link_4_mass" value="0.769" />
-	<property name="link_5_mass" value="0.687" />
-	<!--<property name="link_0_mass" value="0.845" />
-	<property name="link_1_mass" value="0.1" />
-	<property name="link_2_mass" value="0.1" />
-	<property name="link_3_mass" value="0.1" />
-	<property name="link_4_mass" value="0.1" />
-	<property name="link_5_mass" value="0.1" />-->
+	<xacro:property name="link_0_mass" value="0.961" />
+	<xacro:property name="link_1_mass" value="1.390" />
+	<xacro:property name="link_2_mass" value="1.318" />
+	<xacro:property name="link_3_mass" value="0.821" />
+	<xacro:property name="link_4_mass" value="0.769" />
+	<xacro:property name="link_5_mass" value="0.687" />
+	<!--<xacro:property name="link_0_mass" value="0.845" />
+	<xacro:property name="link_1_mass" value="0.1" />
+	<xacro:property name="link_2_mass" value="0.1" />
+	<xacro:property name="link_3_mass" value="0.1" />
+	<xacro:property name="link_4_mass" value="0.1" />
+	<xacro:property name="link_5_mass" value="0.1" />-->
 	<!-- TODO: add inertia tensor-->
 	<xacro:macro name="default_origin">

File: urdf/youbot_base/base.urdf.xacro (robot description, xacro)
@@ -7,30 +7,30 @@
   <xacro:include filename="$(find youbot_description)/urdf/youbot_base/base.transmission.xacro"/>
   <!-- simplified box collision geometry for base -->
-  <property name="base_size_x" value="0.570"/>
-  <property name="base_size_y" value="0.360"/>
-  <property name="base_size_z" value="0.100"/>
-  <property name="base_mass" value="22.0"/>
-  <property name="caster_offset_x" value="0.228"/>
-  <property name="caster_offset_y" value="0.158"/>
-  <property name="caster_offset_z" value="-0.034"/>
-  <property name="caster_mass" value="0.1"/>
-  <property name="wheel_offset_x" value="0.0"/>
-  <property name="wheel_offset_y" value="0.0"/>
-  <property name="wheel_offset_z" value="0.0"/>
-  <property name="wheel_mass" value="1.4"/>
-  <property name="wheel_radius" value="0.0475"/>
-  <property name="wheel_length" value="0.005"/>
-  <property name="caster_joint_damping" value="1.0"/>
-  <property name="caster_joint_friction" value="1.0"/>
-  <property name="caster_joint_effort" value="30"/>
-  <property name="caster_joint_velocity" value="10"/>
-  <property name="caster_joint_safety_k_velocity" value="10.0"/>
-  <property name="wheel_joint_damping" value="1.0"/>
-  <property name="wheel_joint_friction" value="1.0"/>
-  <property name="wheel_joint_effort" value="30"/>
-  <property name="wheel_joint_velocity" value="10"/>
-  <property name="wheel_joint_safety_k_velocity" value="10.0"/>
+  <xacro:property name="base_size_x" value="0.570"/>
+  <xacro:property name="base_size_y" value="0.360"/>
+  <xacro:property name="base_size_z" value="0.100"/>
+  <xacro:property name="base_mass" value="22.0"/>
+  <xacro:property name="caster_offset_x" value="0.228"/>
+  <xacro:property name="caster_offset_y" value="0.158"/>
+  <xacro:property name="caster_offset_z" value="-0.034"/>
+  <xacro:property name="caster_mass" value="0.1"/>
+  <xacro:property name="wheel_offset_x" value="0.0"/>
+  <xacro:property name="wheel_offset_y" value="0.0"/>
+  <xacro:property name="wheel_offset_z" value="0.0"/>
+  <xacro:property name="wheel_mass" value="1.4"/>
+  <xacro:property name="wheel_radius" value="0.0475"/>
+  <xacro:property name="wheel_length" value="0.005"/>
+  <xacro:property name="caster_joint_damping" value="1.0"/>
+  <xacro:property name="caster_joint_friction" value="1.0"/>
+  <xacro:property name="caster_joint_effort" value="30"/>
+  <xacro:property name="caster_joint_velocity" value="10"/>
+  <xacro:property name="caster_joint_safety_k_velocity" value="10.0"/>
+  <xacro:property name="wheel_joint_damping" value="1.0"/>
+  <xacro:property name="wheel_joint_friction" value="1.0"/>
+  <xacro:property name="wheel_joint_effort" value="30"/>
+  <xacro:property name="wheel_joint_velocity" value="10"/>
+  <xacro:property name="wheel_joint_safety_k_velocity" value="10.0"/>
   <xacro:macro name="youbot_base" params="name">
-    <link name="${name}_footprint">
+    <!-- <link name="${name}_footprint">
       <inertial>
         <mass value="0.1"/>
@@ -56,5 +56,5 @@
       <child link="${name}_link"/>
       <parent link="${name}_footprint"/>
-    </joint>
+    </joint>-->
     <link name="${name}_link">
       <inertial>

File: urdf/youbot_gripper/limits.urdf.xacro (robot description, xacro)
@@ -2,8 +2,8 @@
 <robot>
 	<!-- common properties -->
-	<property name="M_PI" value="3.1415926535897931" />
-        <property name="threshold" value="0.001" />
+	<xacro:property name="M_PI" value="3.1415926535897931" />
+        <xacro:property name="threshold" value="0.001" />
 	<!-- fingers limits, values are in meters -->
-	<property name="finger_joint" value="${0.023 / 2.0}" />
-	<property name="finger_joint_soft" value="${(0.023 - threshold) / 2.0}" />
+	<xacro:property name="finger_joint" value="${0.023 / 2.0}" />
+	<xacro:property name="finger_joint_soft" value="${(0.023 - threshold) / 2.0}" />
 </robot>

File: urdf/youbot_plate/plate.urdf.xacro (robot description, xacro)
@@ -7,5 +7,5 @@
 		<!-- joint between arm_7_link and sdh_palm_link -->
 		<joint name="${name}_joint" type="fixed" >
-			<insert_block name="origin" />
+			<xacro:insert_block name="origin" />
 			<parent link="${parent}" />
 			<child link="${name}_link" />
